Commit message: added new 6dof moveit config

File: arc_robot_arm/nodes/arc_robot_arm_urdf.urdf (robot description, URDF)
Before this commit: robot robot_arm_urdf_v1, 8 links, 7 joints
Links:
- link base_link: mass None -> 0.7538944695406217; geometry collision mesh filename=package://arc_robot_arm_urdf_description/meshes/base_link.s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 scale=0.001 0.001 0.001; visual mesh filename=package://arc_robot_arm_urdf_description/meshes/base_link.s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 scale=0.001 0.001 0.001
- link gear1_v1_1: mass None -> 0.028106280846863212; geometry collision mesh filename=package://arc_robot_arm_urdf_description/meshes/gear1_v1_1.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 scale=0.001 0.001 0.001; visual mesh filename=package://arc_robot_arm_urdf_description/meshes/gear1_v1_1.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 scale=0.001 0.001 0.001
- link gear2_v1_1: mass None -> 0.027479876879980724; geometry collision mesh filename=package://arc_robot_arm_urdf_description/meshes/gear2_v1_1.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 scale=0.001 0.001 0.001; visual mesh filename=package://arc_robot_arm_urdf_description/meshes/gear2_v1_1.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 scale=0.001 0.001 0.001
- link gripper_base_v1_1: mass None -> 0.10839935246360793; geometry collision mesh filename=package://arc_robot_arm_urdf_description/meshes/gripper_bas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 scale=0.001 0.001 0.001; visual mesh filename=package://arc_robot_arm_urdf_description/meshes/gripper_bas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 scale=0.001 0.001 0.001
- link link_1_v1_1: mass None -> 0.5341010747394327; geometry collision mesh filename=package://arc_robot_arm_urdf_description/meshes/link_1_v1_1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 scale=0.001 0.001 0.001; visual mesh filename=package://arc_robot_arm_urdf_description/meshes/link_1_v1_1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 scale=0.001 0.001 0.001
- link link_2_v1_1: mass None -> 0.5015278384318742; geometry collision mesh filename=package://arc_robot_arm_urdf_description/meshes/link_2_v1_1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 scale=0.001 0.001 0.001; visual mesh filename=package://arc_robot_arm_urdf_description/meshes/link_2_v1_1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 scale=0.001 0.001 0.001
- link link_3_v1_1: geometry collision mesh filename=package://arc_robot_arm_urdf_description/meshes/link_3_v1_1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 scale=0.001 0.001 0.001; visual mesh filename=package://arc_robot_arm_urdf_description/meshes/link_3_v1_1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 scale=0.001 0.001 0.001
- link link_4_v1_1: mass None -> 0.1295112121194818; geometry collision mesh filename=package://arc_robot_arm_urdf_description/meshes/link_4_v1_1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 scale=0.001 0.001 0.001; visual mesh filename=package://arc_robot_arm_urdf_description/meshes/link_4_v1_1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 scale=0.001 0.001 0.001
Joints:
- joint Rev3: origin xyz=0.033584 0.028776 0.111553 rpy=0 0 0 -> xyz=0.002144 0.00274 0.119949 rpy=0 0 0
- joint Rev4: axis -0.602598 -0.495323 0.625725 -> -0.767993 -0.637134 0.065163; origin xyz=-0.051828 -0.052363 0.052071 rpy=0 0 0 -> xyz=-0.064381 -0.063199 0.000606 rpy=0 0 0
- joint Rev5: axis 0.653959 -0.755876 0.031439 -> 0.639951 -0.767451 0.0385; origin xyz=-0.023741 -0.001146 0.020977 rpy=0 0 0 -> xyz=-0.030336 -0.006739 0.006271 rpy=0 0 0
- joint Rev6: axis -0.188117 -0.122221 0.974512 -> 0.00405 0.053471 0.998561; origin xyz=-0.018773 -0.039683 0.005765 rpy=0 0 0 -> xyz=-0.017687 -0.037266 0.016088 rpy=0 0 0
- joint Rev7: axis -0.188117 -0.122221 0.974512 -> 0.00405 0.053471 0.998561; origin xyz=-0.036364 -0.01935 0.004919 rpy=0 0 0 -> xyz=-0.034902 -0.016622 0.015052 rpy=0 0 0
