Commit message: Add files via upload

File: mvp_arm_6dof_v2_description/urdf/mvp_arm_6dof_v2.xacro (robot description, xacro)
@@ -24,5 +24,5 @@
   </collision>
 </link>
-<link name="old_component__4__1">
+<link name="Servo_Rotator__1__1">
   <inertial>
     <origin rpy="0 0 0" xyz="-0.00016594327411623144 -2.746746623999636e-06 -0.0022433652870559873"/>
@@ -33,5 +33,5 @@
     <origin rpy="0 0 0" xyz="-0.278672 -0.000395 -0.297363"/>
     <geometry>
-      <mesh filename="package://mvp_arm_6dof_v2_description/meshes/old_component__4__1.stl" scale="0.001 0.001 0.001"/>
+      <mesh filename="package://mvp_arm_6dof_v2_description/meshes/Servo_Rotator__1__1.stl" scale="0.001 0.001 0.001"/>
     </geometry>
     <material name="silver"/>
@@ -40,9 +40,9 @@
     <origin rpy="0 0 0" xyz="-0.278672 -0.000395 -0.297363"/>
     <geometry>
-      <mesh filename="package://mvp_arm_6dof_v2_description/meshes/old_component__4__1.stl" scale="0.001 0.001 0.001"/>
-    </geometry>
-  </collision>
-</link>
-<link name="old_component__6__1">
+      <mesh filename="package://mvp_arm_6dof_v2_description/meshes/Servo_Rotator__1__1.stl" scale="0.001 0.001 0.001"/>
+    </geometry>
+  </collision>
+</link>
+<link name="Servo_Rotator__2__1">
   <inertial>
     <origin rpy="0 0 0" xyz="-1.9052915553596783e-07 -0.0022492646837299415 2.4533432791407073e-06"/>
@@ -53,5 +53,5 @@
     <origin rpy="0 0 0" xyz="-0.222902 0.015475 -0.385928"/>
     <geometry>
-      <mesh filename="package://mvp_arm_6dof_v2_description/meshes/old_component__6__1.stl" scale="0.001 0.001 0.001"/>
+      <mesh filename="package://mvp_arm_6dof_v2_description/meshes/Servo_Rotator__2__1.stl" scale="0.001 0.001 0.001"/>
     </geometry>
     <material name="silver"/>
@@ -60,9 +60,9 @@
     <origin rpy="0 0 0" xyz="-0.222902 0.015475 -0.385928"/>
     <geometry>
-      <mesh filename="package://mvp_arm_6dof_v2_description/meshes/old_component__6__1.stl" scale="0.001 0.001 0.001"/>
-    </geometry>
-  </collision>
-</link>
-<link name="old_component__7__1">
+      <mesh filename="package://mvp_arm_6dof_v2_description/meshes/Servo_Rotator__2__1.stl" scale="0.001 0.001 0.001"/>
+    </geometry>
+  </collision>
+</link>
+<link name="Servo__3__1">
   <inertial>
     <origin rpy="0 0 0" xyz="0.022878488280711123 0.015454485443440637 -0.008032933007486143"/>
@@ -73,5 +73,5 @@
     <origin rpy="0 0 0" xyz="-0.186907 0.015215 -0.393949"/>
     <geometry>
-      <mesh filename="package://mvp_arm_6dof_v2_description/meshes/old_component__7__1.stl" scale="0.001 0.001 0.001"/>
+      <mesh filename="package://mvp_arm_6dof_v2_description/meshes/Servo__3__1.stl" scale="0.001 0.001 0.001"/>
     </geometry>
     <material name="silver"/>
@@ -80,9 +80,9 @@
     <origin rpy="0 0 0" xyz="-0.186907 0.015215 -0.393949"/>
     <geometry>
-      <mesh filename="package://mvp_arm_6dof_v2_description/meshes/old_component__7__1.stl" scale="0.001 0.001 0.001"/>
-    </geometry>
-  </collision>
-</link>
-<link name="old_component__9__1">
+      <mesh filename="package://mvp_arm_6dof_v2_description/meshes/Servo__3__1.stl" scale="0.001 0.001 0.001"/>
+    </geometry>
+  </collision>
+</link>
+<link name="Servo__2__1">
   <inertial>
     <origin rpy="0 0 0" xyz="-0.0182436166094693 -0.008545149871361533 -0.018077639575404758"/>
@@ -93,5 +93,5 @@
     <origin rpy="0 0 0" xyz="-0.23753 -0.00898 -0.34922"/>
     <geometry>
-      <mesh filename="package://mvp_arm_6dof_v2_description/meshes/old_component__9__1.stl" scale="0.001 0.001 0.001"/>
+      <mesh filename="package://mvp_arm_6dof_v2_description/meshes/Servo__2__1.stl" scale="0.001 0.001 0.001"/>
     </geometry>
     <material name="silver"/>
@@ -100,9 +100,9 @@
     <origin rpy="0 0 0" xyz="-0.23753 -0.00898 -0.34922"/>
     <geometry>
-      <mesh filename="package://mvp_arm_6dof_v2_description/meshes/old_component__9__1.stl" scale="0.001 0.001 0.001"/>
-    </geometry>
-  </collision>
-</link>
-<link name="old_component__10__1">
+      <mesh filename="package://mvp_arm_6dof_v2_description/meshes/Servo__2__1.stl" scale="0.001 0.001 0.001"/>
+    </geometry>
+  </collision>
+</link>
+<link name="Servo_Rotator__3__1">
   <inertial>
     <origin rpy="0 0 0" xyz="0.002243165392088464 2.5336489333719747e-07 -0.00016573648369289096"/>
@@ -113,5 +113,5 @@
     <origin rpy="0 0 0" xyz="-0.233991 -0.000418 -0.316903"/>
     <geometry>
-      <mesh filename="package://mvp_arm_6dof_v2_description/meshes/old_component__10__1.stl" scale="0.001 0.001 0.001"/>
+      <mesh filename="package://mvp_arm_6dof_v2_description/meshes/Servo_Rotator__3__1.stl" scale="0.001 0.001 0.001"/>
     </geometry>
     <material name="silver"/>
@@ -120,9 +120,9 @@
     <origin rpy="0 0 0" xyz="-0.233991 -0.000418 -0.316903"/>
     <geometry>
-      <mesh filename="package://mvp_arm_6dof_v2_description/meshes/old_component__10__1.stl" scale="0.001 0.001 0.001"/>
-    </geometry>
-  </collision>
-</link>
-<link name="old_component__12__1">
+      <mesh filename="package://mvp_arm_6dof_v2_description/meshes/Servo_Rotator__3__1.stl" scale="0.001 0.001 0.001"/>
+    </geometry>
+  </collision>
+</link>
+<link name="Servo__4__1">
   <inertial>
     <origin rpy="0 0 0" xyz="0.015722336863971474 -1.2746670361859992e-05 0.013106406607165055"/>
@@ -133,5 +133,5 @@
     <origin rpy="0 0 0" xyz="-0.033133 -0.000807 -0.354024"/>
     <geometry>
-      <mesh filename="package://mvp_arm_6dof_v2_description/meshes/old_component__12__1.stl" scale="0.001 0.001 0.001"/>
+      <mesh filename="package://mvp_arm_6dof_v2_description/meshes/Servo__4__1.stl" scale="0.001 0.001 0.001"/>
     </geometry>
     <material name="silver"/>
@@ -140,9 +140,9 @@
     <origin rpy="0 0 0" xyz="-0.033133 -0.000807 -0.354024"/>
     <geometry>
-      <mesh filename="package://mvp_arm_6dof_v2_description/meshes/old_component__12__1.stl" scale="0.001 0.001 0.001"/>
-    </geometry>
-  </collision>
-</link>
-<link name="old_component__3__1">
+      <mesh filename="package://mvp_arm_6dof_v2_description/meshes/Servo__4__1.stl" scale="0.001 0.001 0.001"/>
+    </geometry>
+  </collision>
+</link>
+<link name="Bracket__3__1">
   <inertial>
     <origin rpy="0 0 0" xyz="0.016001488175731965 -0.008003232726281992 0.003640364466268753"/>
@@ -153,5 +153,5 @@
     <origin rpy="0 0 0" xyz="-0.033405 -0.00877 -0.390032"/>
     <geometry>
-      <mesh filename="package://mvp_arm_6dof_v2_description/meshes/old_component__3__1.stl" scale="0.001 0.001 0.001"/>
+      <mesh filename="package://mvp_arm_6dof_v2_description/meshes/Bracket__3__1.stl" scale="0.001 0.001 0.001"/>
     </geometry>
     <material name="silver"/>
@@ -160,9 +160,9 @@
     <origin rpy="0 0 0" xyz="-0.033405 -0.00877 -0.390032"/>
     <geometry>
-      <mesh filename="package://mvp_arm_6dof_v2_description/meshes/old_component__3__1.stl" scale="0.001 0.001 0.001"/>
-    </geometry>
-  </collision>
-</link>
-<link name="old_component__11__1">
+      <mesh filename="package://mvp_arm_6dof_v2_description/meshes/Bracket__3__1.stl" scale="0.001 0.001 0.001"/>
+    </geometry>
+  </collision>
+</link>
+<link name="Servo_Rotator__4__1">
   <inertial>
     <origin rpy="0 0 0" xyz="0.0022555945146578715 -2.6497304426618355e-07 0.007999036398771475"/>
@@ -173,5 +173,5 @@
     <origin rpy="0 0 0" xyz="-0.028628 -0.000807 -0.346026"/>
     <geometry>
-      <mesh filename="package://mvp_arm_6dof_v2_description/meshes/old_component__11__1.stl" scale="0.001 0.001 0.001"/>
+      <mesh filename="package://mvp_arm_6dof_v2_description/meshes/Servo_Rotator__4__1.stl" scale="0.001 0.001 0.001"/>
     </geometry>
     <material name="silver"/>
@@ -180,9 +180,9 @@
     <origin rpy="0 0 0" xyz="-0.028628 -0.000807 -0.346026"/>
     <geometry>
-      <mesh filename="package://mvp_arm_6dof_v2_description/meshes/old_component__11__1.stl" scale="0.001 0.001 0.001"/>
-    </geometry>
-  </collision>
-</link>
-<link name="old_component__15__1">
+      <mesh filename="package://mvp_arm_6dof_v2_description/meshes/Servo_Rotator__4__1.stl" scale="0.001 0.001 0.001"/>
+    </geometry>
+  </collision>
+</link>
+<link name="Servo__5__1">
   <inertial>
     <origin rpy="0 0 0" xyz="0.013116173460706801 -0.01571500032507959 -9.058538409600914e-06"/>
@@ -193,5 +193,5 @@
     <origin rpy="0 0 0" xyz="0.012867 -0.017 -0.354052"/>
     <geometry>
-      <mesh filename="package://mvp_arm_6dof_v2_description/meshes/old_component__15__1.stl" scale="0.001 0.001 0.001"/>
+      <mesh filename="package://mvp_arm_6dof_v2_description/meshes/Servo__5__1.stl" scale="0.001 0.001 0.001"/>
     </geometry>
     <material name="silver"/>
@@ -200,9 +200,9 @@
     <origin rpy="0 0 0" xyz="0.012867 -0.017 -0.354052"/>
     <geometry>
-      <mesh filename="package://mvp_arm_6dof_v2_description/meshes/old_component__15__1.stl" scale="0.001 0.001 0.001"/>
-    </geometry>
-  </collision>
-</link>
-<link name="old_component__13__1">
+      <mesh filename="package://mvp_arm_6dof_v2_description/meshes/Servo__5__1.stl" scale="0.001 0.001 0.001"/>
+    </geometry>
+  </collision>
+</link>
+<link name="Bracket__5__1">
   <inertial>
     <origin rpy="0 0 0" xyz="0.0036634715521508127 0.01599973502692581 0.007997526572222857"/>
@@ -213,5 +213,5 @@
     <origin rpy="0 0 0" xyz="-0.023128 0.015193 -0.34603"/>
     <geometry>
-      <mesh filename="package://mvp_arm_6dof_v2_description/meshes/old_component__13__1.stl" scale="0.001 0.001 0.001"/>
+      <mesh filename="package://mvp_arm_6dof_v2_description/meshes/Bracket__5__1.stl" scale="0.001 0.001 0.001"/>
     </geometry>
     <material name="silver"/>
@@ -220,9 +220,9 @@
     <origin rpy="0 0 0" xyz="-0.023128 0.015193 -0.34603"/>
     <geometry>
-      <mesh filename="package://mvp_arm_6dof_v2_description/meshes/old_component__13__1.stl" scale="0.001 0.001 0.001"/>
-    </geometry>
-  </collision>
-</link>
-<link name="old_component__20__1">
+      <mesh filename="package://mvp_arm_6dof_v2_description/meshes/Bracket__5__1.stl" scale="0.001 0.001 0.001"/>
+    </geometry>
+  </collision>
+</link>
+<link name="Forearm_1">
   <inertial>
     <origin rpy="0 0 0" xyz="0.048128469775268856 4.4527298823126334e-07 -6.254652134507488e-05"/>
@@ -233,5 +233,5 @@
     <origin rpy="0 0 0" xyz="-0.081402 -0.000774 -0.385994"/>
     <geometry>
-      <mesh filename="package://mvp_arm_6dof_v2_description/meshes/old_component__20__1.stl" scale="0.001 0.001 0.001"/>
+      <mesh filename="package://mvp_arm_6dof_v2_description/meshes/Forearm_1.stl" scale="0.001 0.001 0.001"/>
     </geometry>
     <material name="silver"/>
@@ -240,9 +240,9 @@
     <origin rpy="0 0 0" xyz="-0.081402 -0.000774 -0.385994"/>
     <geometry>
-      <mesh filename="package://mvp_arm_6dof_v2_description/meshes/old_component__20__1.stl" scale="0.001 0.001 0.001"/>
-    </geometry>
-  </collision>
-</link>
-<link name="old_component__18__1">
+      <mesh filename="package://mvp_arm_6dof_v2_description/meshes/Forearm_1.stl" scale="0.001 0.001 0.001"/>
+    </geometry>
+  </collision>
+</link>
+<link name="Forearm_Joint_1">
   <inertial>
     <origin rpy="0 0 0" xyz="0.019545111524890385 7.79105773380162e-06 -0.00783005977281992"/>
@@ -253,5 +253,5 @@
     <origin rpy="0 0 0" xyz="-0.041408 -0.000765 -0.395519"/>
     <geometry>
-      <mesh filename="package://mvp_arm_6dof_v2_description/meshes/old_component__18__1.stl" scale="0.001 0.001 0.001"/>
+      <mesh filename="package://mvp_arm_6dof_v2_description/meshes/Forearm_Joint_1.stl" scale="0.001 0.001 0.001"/>
     </geometry>
     <material name="silver"/>
@@ -260,9 +260,9 @@
     <origin rpy="0 0 0" xyz="-0.041408 -0.000765 -0.395519"/>
     <geometry>
-      <mesh filename="package://mvp_arm_6dof_v2_description/meshes/old_component__18__1.stl" scale="0.001 0.001 0.001"/>
-    </geometry>
-  </collision>
-</link>
-<link name="old_component__14__1">
+      <mesh filename="package://mvp_arm_6dof_v2_description/meshes/Forearm_Joint_1.stl" scale="0.001 0.001 0.001"/>
+    </geometry>
+  </collision>
+</link>
+<link name="Servo_Rotator__5__1">
   <inertial>
     <origin rpy="0 0 0" xyz="0.00799986632219811 -0.002251236293083818 -5.340036253298486e-06"/>
@@ -273,5 +273,5 @@
     <origin rpy="0 0 0" xyz="0.020867 -0.0215 -0.354057"/>
     <geometry>
-      <mesh filename="package://mvp_arm_6dof_v2_description/meshes/old_component__14__1.stl" scale="0.001 0.001 0.001"/>
+      <mesh filename="package://mvp_arm_6dof_v2_description/meshes/Servo_Rotator__5__1.stl" scale="0.001 0.001 0.001"/>
     </geometry>
     <material name="silver"/>
@@ -280,9 +280,9 @@
     <origin rpy="0 0 0" xyz="0.020867 -0.0215 -0.354057"/>
     <geometry>
-      <mesh filename="package://mvp_arm_6dof_v2_description/meshes/old_component__14__1.stl" scale="0.001 0.001 0.001"/>
-    </geometry>
-  </collision>
-</link>
-<link name="old_component__16__2">
+      <mesh filename="package://mvp_arm_6dof_v2_description/meshes/Servo_Rotator__5__1.stl" scale="0.001 0.001 0.001"/>
+    </geometry>
+  </collision>
+</link>
+<link name="Elbow_Hinge__1__2">
   <inertial>
     <origin rpy="0 0 0" xyz="-0.013495411982010678 3.3022629769563494e-15 0.010254437334501432"/>
@@ -293,5 +293,5 @@
     <origin rpy="0 0 0" xyz="-0.000617 -0.0005 -0.327543"/>
     <geometry>
-      <mesh filename="package://mvp_arm_6dof_v2_description/meshes/old_component__16__2.stl" scale="0.001 0.001 0.001"/>
+      <mesh filename="package://mvp_arm_6dof_v2_description/meshes/Elbow_Hinge__1__2.stl" scale="0.001 0.001 0.001"/>
     </geometry>
     <material name="silver"/>
@@ -300,9 +300,9 @@
     <origin rpy="0 0 0" xyz="-0.000617 -0.0005 -0.327543"/>
     <geometry>
-      <mesh filename="package://mvp_arm_6dof_v2_description/meshes/old_component__16__2.stl" scale="0.001 0.001 0.001"/>
-    </geometry>
-  </collision>
-</link>
-<link name="old_component__17__1">
+      <mesh filename="package://mvp_arm_6dof_v2_description/meshes/Elbow_Hinge__1__2.stl" scale="0.001 0.001 0.001"/>
+    </geometry>
+  </collision>
+</link>
+<link name="Arm_Link_1">
   <inertial>
     <origin rpy="0 0 0" xyz="4.7314773535239024e-05 -0.018999999999999035 0.07720570491989823"/>
@@ -313,5 +313,5 @@
     <origin rpy="0 0 0" xyz="0.011984 -0.0195 -0.162551"/>
     <geometry>
-      <mesh filename="package://mvp_arm_6dof_v2_description/meshes/old_component__17__1.stl" scale="0.001 0.001 0.001"/>
+      <mesh filename="package://mvp_arm_6dof_v2_description/meshes/Arm_Link_1.stl" scale="0.001 0.001 0.001"/>
     </geometry>
     <material name="silver"/>
@@ -320,9 +320,9 @@
     <origin rpy="0 0 0" xyz="0.011984 -0.0195 -0.162551"/>
     <geometry>
-      <mesh filename="package://mvp_arm_6dof_v2_description/meshes/old_component__17__1.stl" scale="0.001 0.001 0.001"/>
-    </geometry>
-  </collision>
-</link>
-<link name="old_component__21__1">
+      <mesh filename="package://mvp_arm_6dof_v2_description/meshes/Arm_Link_1.stl" scale="0.001 0.001 0.001"/>
+    </geometry>
+  </collision>
+</link>
+<link name="Shoulder_Joint_1">
   <inertial>
     <origin rpy="0 0 0" xyz="7.287449404962842e-05 0.0016854028904963768 0.013016506375220449"/>
@@ -333,5 +333,5 @@
     <origin rpy="0 0 0" xyz="0.0 -0.0 -0.131"/>
     <geometry>
-      <mesh filename="package://mvp_arm_6dof_v2_description/meshes/old_component__21__1.stl" scale="0.001 0.001 0.001"/>
+      <mesh filename="package://mvp_arm_6dof_v2_description/meshes/Shoulder_Joint_1.stl" scale="0.001 0.001 0.001"/>
     </geometry>
     <material name="silver"/>
@@ -340,9 +340,9 @@
     <origin rpy="0 0 0" xyz="0.0 -0.0 -0.131"/>
     <geometry>
-      <mesh filename="package://mvp_arm_6dof_v2_description/meshes/old_component__21__1.stl" scale="0.001 0.001 0.001"/>
-    </geometry>
-  </collision>
-</link>
-<link name="old_component__22__1">
+      <mesh filename="package://mvp_arm_6dof_v2_description/meshes/Shoulder_Joint_1.stl" scale="0.001 0.001 0.001"/>
+    </geometry>
+  </collision>
+</link>
+<link name="Wrist_Hinge_1">
   <inertial>
     <origin rpy="0 0 0" xyz="-0.0006100381163169633 0.020989965286603927 -0.008256993530336987"/>
@@ -353,5 +353,5 @@
     <origin rpy="0 0 0" xyz="-0.222312 0.019985 -0.377955"/>
     <geometry>
-      <mesh filename="package://mvp_arm_6dof_v2_description/meshes/old_component__22__1.stl" scale="0.001 0.001 0.001"/>
+      <mesh filename="package://mvp_arm_6dof_v2_description/meshes/Wrist_Hinge_1.stl" scale="0.001 0.001 0.001"/>
     </geometry>
     <material name="silver"/>
@@ -360,9 +360,9 @@
     <origin rpy="0 0 0" xyz="-0.222312 0.019985 -0.377955"/>
     <geometry>
-      <mesh filename="package://mvp_arm_6dof_v2_description/meshes/old_component__22__1.stl" scale="0.001 0.001 0.001"/>
-    </geometry>
-  </collision>
-</link>
-<link name="old_component__1__1">
+      <mesh filename="package://mvp_arm_6dof_v2_description/meshes/Wrist_Hinge_1.stl" scale="0.001 0.001 0.001"/>
+    </geometry>
+  </collision>
+</link>
+<link name="Bracket__1__1">
   <inertial>
     <origin rpy="0 0 0" xyz="0.0024261508410601262 9.893036074812322e-06 0.007842544811764884"/>
@@ -373,5 +373,5 @@
     <origin rpy="0 0 0" xyz="-0.237889 -0.000408 -0.308593"/>
     <geometry>
-      <mesh filename="package://mvp_arm_6dof_v2_description/meshes/old_component__1__1.stl" scale="0.001 0.001 0.001"/>
+      <mesh filename="package://mvp_arm_6dof_v2_description/meshes/Bracket__1__1.stl" scale="0.001 0.001 0.001"/>
     </geometry>
     <material name="silver"/>
@@ -380,9 +380,9 @@
     <origin rpy="0 0 0" xyz="-0.237889 -0.000408 -0.308593"/>
     <geometry>
-      <mesh filename="package://mvp_arm_6dof_v2_description/meshes/old_component__1__1.stl" scale="0.001 0.001 0.001"/>
-    </geometry>
-  </collision>
-</link>
-<link name="old_component__5__1">
+      <mesh filename="package://mvp_arm_6dof_v2_description/meshes/Bracket__1__1.stl" scale="0.001 0.001 0.001"/>
+    </geometry>
+  </collision>
+</link>
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