Commit message: updated 6dof robot description with gripper

File: mvp_arm_6dof_v2_description/urdf/mvp_arm_6dof_v2.xacro (robot description, xacro)
@@ -6,7 +6,7 @@
 <link name="base_link">
   <inertial>
-    <origin rpy="0 0 0" xyz="5.2381743387286404e-12 0.0006676510153735648 0.09744738648290209"/>
+    <origin rpy="0 0 0" xyz="-0.0002685563857322659 -0.004117383840236073 0.09720599739360383"/>
     <mass value="0.2255222028913783"/>
-    <inertia ixx="0.000624" ixy="0.0" ixz="0.0" iyy="0.000615" iyz="1e-06" izz="0.001121"/>
+    <inertia ixx="0.000625" ixy="-0.0" ixz="-1.3e-05" iyy="0.000615" iyz="0.0" izz="0.001121"/>
   </inertial>
   <visual>
@@ -26,10 +26,10 @@
 <link name="Servo_Rotator__1__1">
   <inertial>
-    <origin rpy="0 0 0" xyz="-0.00016594327411623144 -2.746746623999636e-06 -0.0022433652870559873"/>
+    <origin rpy="0 0 0" xyz="4.696790787805938e-05 2.736599626973436e-05 -0.0022484802383110902"/>
     <mass value="0.012286224598738087"/>
-    <inertia ixx="0.0" ixy="0.0" ixz="0.0" iyy="0.0" iyz="0.0" izz="1e-06"/>
-  </inertial>
-  <visual>
-    <origin rpy="0 0 0" xyz="-0.278672 -0.000395 -0.297363"/>
+    <inertia ixx="0.0" ixy="0.0" ixz="-0.0" iyy="0.0" iyz="-0.0" izz="1e-06"/>
+  </inertial>
+  <visual>
+    <origin rpy="0 0 0" xyz="-0.278678 0.002272 -0.30869"/>
     <geometry>
       <mesh filename="package://mvp_arm_6dof_v2_description/meshes/Servo_Rotator__1__1.stl" scale="0.001 0.001 0.001"/>
@@ -38,5 +38,5 @@
   </visual>
   <collision>
-    <origin rpy="0 0 0" xyz="-0.278672 -0.000395 -0.297363"/>
+    <origin rpy="0 0 0" xyz="-0.278678 0.002272 -0.30869"/>
     <geometry>
       <mesh filename="package://mvp_arm_6dof_v2_description/meshes/Servo_Rotator__1__1.stl" scale="0.001 0.001 0.001"/>
@@ -46,10 +46,10 @@
 <link name="Servo_Rotator__2__1">
   <inertial>
-    <origin rpy="0 0 0" xyz="-1.9052915553596783e-07 -0.0022492646837299415 2.4533432791407073e-06"/>
+    <origin rpy="0 0 0" xyz="3.197445282709932e-07 -0.002249396881839328 1.0236701699029016e-05"/>
     <mass value="0.012286224598738087"/>
     <inertia ixx="0.0" ixy="-0.0" ixz="0.0" iyy="1e-06" iyz="-0.0" izz="0.0"/>
   </inertial>
   <visual>
-    <origin rpy="0 0 0" xyz="-0.222902 0.015475 -0.385928"/>
+    <origin rpy="0 0 0" xyz="-0.214785 0.018149 -0.391636"/>
     <geometry>
       <mesh filename="package://mvp_arm_6dof_v2_description/meshes/Servo_Rotator__2__1.stl" scale="0.001 0.001 0.001"/>
@@ -58,5 +58,5 @@
   </visual>
   <collision>
-    <origin rpy="0 0 0" xyz="-0.222902 0.015475 -0.385928"/>
+    <origin rpy="0 0 0" xyz="-0.214785 0.018149 -0.391636"/>
     <geometry>
       <mesh filename="package://mvp_arm_6dof_v2_description/meshes/Servo_Rotator__2__1.stl" scale="0.001 0.001 0.001"/>
@@ -66,10 +66,10 @@
 <link name="Servo__3__1">
   <inertial>
-    <origin rpy="0 0 0" xyz="0.022878488280711123 0.015454485443440637 -0.008032933007486143"/>
+    <origin rpy="0 0 0" xyz="0.023084439447248556 0.01543302398482891 -0.007466520807867916"/>
     <mass value="0.32411536495008075"/>
-    <inertia ixx="5e-05" ixy="-2e-06" ixz="0.0" iyy="7.9e-05" iyz="0.0" izz="9.1e-05"/>
-  </inertial>
-  <visual>
-    <origin rpy="0 0 0" xyz="-0.186907 0.015215 -0.393949"/>
+    <inertia ixx="5e-05" ixy="-2e-06" ixz="-1e-06" iyy="7.9e-05" iyz="0.0" izz="9.1e-05"/>
+  </inertial>
+  <visual>
+    <origin rpy="0 0 0" xyz="-0.178587 0.017871 -0.398684"/>
     <geometry>
       <mesh filename="package://mvp_arm_6dof_v2_description/meshes/Servo__3__1.stl" scale="0.001 0.001 0.001"/>
@@ -78,5 +78,5 @@
   </visual>
   <collision>
-    <origin rpy="0 0 0" xyz="-0.186907 0.015215 -0.393949"/>
+    <origin rpy="0 0 0" xyz="-0.178587 0.017871 -0.398684"/>
     <geometry>
       <mesh filename="package://mvp_arm_6dof_v2_description/meshes/Servo__3__1.stl" scale="0.001 0.001 0.001"/>
@@ -86,10 +86,10 @@
 <link name="Servo__2__1">
   <inertial>
-    <origin rpy="0 0 0" xyz="-0.0182436166094693 -0.008545149871361533 -0.018077639575404758"/>
+    <origin rpy="0 0 0" xyz="-0.01645020938837613 -0.008616049568100454 -0.0196927644624752"/>
     <mass value="0.32411536495008075"/>
-    <inertia ixx="7.9e-05" ixy="0.0" ixz="-4e-06" iyy="9.1e-05" iyz="-0.0" izz="5e-05"/>
-  </inertial>
-  <visual>
-    <origin rpy="0 0 0" xyz="-0.23753 -0.00898 -0.34922"/>
+    <inertia ixx="7.9e-05" ixy="0.0" ixz="-1e-06" iyy="9.1e-05" iyz="-0.0" izz="5e-05"/>
+  </inertial>
+  <visual>
+    <origin rpy="0 0 0" xyz="-0.232814 -0.00619 -0.356393"/>
     <geometry>
       <mesh filename="package://mvp_arm_6dof_v2_description/meshes/Servo__2__1.stl" scale="0.001 0.001 0.001"/>
@@ -98,5 +98,5 @@
   </visual>
   <collision>
-    <origin rpy="0 0 0" xyz="-0.23753 -0.00898 -0.34922"/>
+    <origin rpy="0 0 0" xyz="-0.232814 -0.00619 -0.356393"/>
     <geometry>
       <mesh filename="package://mvp_arm_6dof_v2_description/meshes/Servo__2__1.stl" scale="0.001 0.001 0.001"/>
@@ -106,10 +106,10 @@
 <link name="Servo_Rotator__3__1">
   <inertial>
-    <origin rpy="0 0 0" xyz="0.002243165392088464 2.5336489333719747e-07 -0.00016573648369289096"/>
+    <origin rpy="0 0 0" xyz="0.002249048184267688 1.7890290807034276e-07 4.676532271863376e-05"/>
     <mass value="0.012286224598738087"/>
-    <inertia ixx="1e-06" ixy="-0.0" ixz="-0.0" iyy="0.0" iyz="0.0" izz="0.0"/>
-  </inertial>
-  <visual>
-    <origin rpy="0 0 0" xyz="-0.233991 -0.000418 -0.316903"/>
+    <inertia ixx="1e-06" ixy="0.0" ixz="0.0" iyy="0.0" iyz="0.0" izz="0.0"/>
+  </inertial>
+  <visual>
+    <origin rpy="0 0 0" xyz="-0.232349 0.002482 -0.323916"/>
     <geometry>
       <mesh filename="package://mvp_arm_6dof_v2_description/meshes/Servo_Rotator__3__1.stl" scale="0.001 0.001 0.001"/>
@@ -118,5 +118,5 @@
   </visual>
   <collision>
-    <origin rpy="0 0 0" xyz="-0.233991 -0.000418 -0.316903"/>
+    <origin rpy="0 0 0" xyz="-0.232349 0.002482 -0.323916"/>
     <geometry>
       <mesh filename="package://mvp_arm_6dof_v2_description/meshes/Servo_Rotator__3__1.stl" scale="0.001 0.001 0.001"/>
@@ -126,10 +126,10 @@
 <link name="Servo__4__1">
   <inertial>
-    <origin rpy="0 0 0" xyz="0.015722336863971474 -1.2746670361859992e-05 0.013106406607165055"/>
+    <origin rpy="0 0 0" xyz="0.015363533740432825 3.599470012234868e-05 0.01352566905944469"/>
     <mass value="0.32411536495008075"/>
-    <inertia ixx="7.9e-05" ixy="0.0" ixz="1e-06" iyy="9.1e-05" iyz="0.0" izz="5e-05"/>
-  </inertial>
-  <visual>
-    <origin rpy="0 0 0" xyz="-0.033133 -0.000807 -0.354024"/>
+    <inertia ixx="7.9e-05" ixy="0.0" ixz="2e-06" iyy="9.1e-05" iyz="-0.0" izz="5e-05"/>
+  </inertial>
+  <visual>
+    <origin rpy="0 0 0" xyz="-0.025942 0.002022 -0.354577"/>
     <geometry>
       <mesh filename="package://mvp_arm_6dof_v2_description/meshes/Servo__4__1.stl" scale="0.001 0.001 0.001"/>
@@ -138,5 +138,5 @@
   </visual>
   <collision>
-    <origin rpy="0 0 0" xyz="-0.033133 -0.000807 -0.354024"/>
+    <origin rpy="0 0 0" xyz="-0.025942 0.002022 -0.354577"/>
     <geometry>
       <mesh filename="package://mvp_arm_6dof_v2_description/meshes/Servo__4__1.stl" scale="0.001 0.001 0.001"/>
@@ -146,10 +146,10 @@
 <link name="Bracket__3__1">
   <inertial>
-    <origin rpy="0 0 0" xyz="0.016001488175731965 -0.008003232726281992 0.003640364466268753"/>
+    <origin rpy="0 0 0" xyz="0.01589864118251931 -0.007987181894295325 0.004097782701024066"/>
     <mass value="0.0016262220015435807"/>
-    <inertia ixx="0.0" ixy="-0.0" ixz="0.0" iyy="0.0" iyz="-0.0" izz="0.0"/>
-  </inertial>
-  <visual>
-    <origin rpy="0 0 0" xyz="-0.033405 -0.00877 -0.390032"/>
+    <inertia ixx="0.0" ixy="-0.0" ixz="-0.0" iyy="0.0" iyz="0.0" izz="0.0"/>
+  </inertial>
+  <visual>
+    <origin rpy="0 0 0" xyz="-0.025243 -0.006064 -0.390552"/>
     <geometry>
       <mesh filename="package://mvp_arm_6dof_v2_description/meshes/Bracket__3__1.stl" scale="0.001 0.001 0.001"/>
@@ -158,5 +158,5 @@
   </visual>
   <collision>
-    <origin rpy="0 0 0" xyz="-0.033405 -0.00877 -0.390032"/>
+    <origin rpy="0 0 0" xyz="-0.025243 -0.006064 -0.390552"/>
     <geometry>
       <mesh filename="package://mvp_arm_6dof_v2_description/meshes/Bracket__3__1.stl" scale="0.001 0.001 0.001"/>
@@ -166,10 +166,10 @@
 <link name="Servo_Rotator__4__1">
   <inertial>
-    <origin rpy="0 0 0" xyz="0.0022555945146578715 -2.6497304426618355e-07 0.007999036398771475"/>
+    <origin rpy="0 0 0" xyz="0.0020392727454433754 1.9599116875569037e-05 0.008056069500829488"/>
     <mass value="0.012286224598738087"/>
-    <inertia ixx="1e-06" ixy="0.0" ixz="-0.0" iyy="0.0" iyz="0.0" izz="0.0"/>
-  </inertial>
-  <visual>
-    <origin rpy="0 0 0" xyz="-0.028628 -0.000807 -0.346026"/>
+    <inertia ixx="1e-06" ixy="0.0" ixz="0.0" iyy="0.0" iyz="0.0" izz="0.0"/>
+  </inertial>
+  <visual>
+    <origin rpy="0 0 0" xyz="-0.021654 0.002042 -0.346462"/>
     <geometry>
       <mesh filename="package://mvp_arm_6dof_v2_description/meshes/Servo_Rotator__4__1.stl" scale="0.001 0.001 0.001"/>
@@ -178,5 +178,5 @@
   </visual>
   <collision>
-    <origin rpy="0 0 0" xyz="-0.028628 -0.000807 -0.346026"/>
+    <origin rpy="0 0 0" xyz="-0.021654 0.002042 -0.346462"/>
     <geometry>
       <mesh filename="package://mvp_arm_6dof_v2_description/meshes/Servo_Rotator__4__1.stl" scale="0.001 0.001 0.001"/>
@@ -186,10 +186,10 @@
 <link name="Servo__5__1">
   <inertial>
-    <origin rpy="0 0 0" xyz="0.013116173460706801 -0.01571500032507959 -9.058538409600914e-06"/>
+    <origin rpy="0 0 0" xyz="0.013114397820069863 -0.015711494309324826 0.0003817734354029101"/>
     <mass value="0.32411536495008075"/>
-    <inertia ixx="5e-05" ixy="-2e-06" ixz="0.0" iyy="7.9e-05" iyz="0.0" izz="9.1e-05"/>
-  </inertial>
-  <visual>
-    <origin rpy="0 0 0" xyz="0.012867 -0.017 -0.354052"/>
+    <inertia ixx="5e-05" ixy="-2e-06" ixz="-1e-06" iyy="7.9e-05" iyz="-0.0" izz="9.1e-05"/>
+  </inertial>
+  <visual>
+    <origin rpy="0 0 0" xyz="0.020045 -0.01416 -0.353328"/>
     <geometry>
       <mesh filename="package://mvp_arm_6dof_v2_description/meshes/Servo__5__1.stl" scale="0.001 0.001 0.001"/>
@@ -198,5 +198,5 @@
   </visual>
   <collision>
-    <origin rpy="0 0 0" xyz="0.012867 -0.017 -0.354052"/>
+    <origin rpy="0 0 0" xyz="0.020045 -0.01416 -0.353328"/>
     <geometry>
       <mesh filename="package://mvp_arm_6dof_v2_description/meshes/Servo__5__1.stl" scale="0.001 0.001 0.001"/>
@@ -206,210 +206,210 @@
 <link name="Bracket__5__1">
   <inertial>
-    <origin rpy="0 0 0" xyz="0.0036634715521508127 0.01599973502692581 0.007997526572222857"/>
-    <mass value="0.0016262220015435807"/>
-    <inertia ixx="0.0" ixy="0.0" ixz="-0.0" iyy="0.0" iyz="0.0" izz="0.0"/>
-  </inertial>
-  <visual>
-    <origin rpy="0 0 0" xyz="-0.023128 0.015193 -0.34603"/>
-    <geometry>
-      <mesh filename="package://mvp_arm_6dof_v2_description/meshes/Bracket__5__1.stl" scale="0.001 0.001 0.001"/>
-    </geometry>
-    <material name="silver"/>
-  </visual>
-  <collision>
-    <origin rpy="0 0 0" xyz="-0.023128 0.015193 -0.34603"/>
-    <geometry>
-      <mesh filename="package://mvp_arm_6dof_v2_description/meshes/Bracket__5__1.stl" scale="0.001 0.001 0.001"/>
-    </geometry>
-  </collision>
-</link>
-<link name="Forearm_1">
-  <inertial>
-    <origin rpy="0 0 0" xyz="0.048128469775268856 4.4527298823126334e-07 -6.254652134507488e-05"/>
-    <mass value="0.7719250888938243"/>
-    <inertia ixx="0.000141" ixy="-0.0" ixz="-1e-06" iyy="0.000726" iyz="0.0" izz="0.000771"/>
-  </inertial>
-  <visual>
-    <origin rpy="0 0 0" xyz="-0.081402 -0.000774 -0.385994"/>
-    <geometry>
-      <mesh filename="package://mvp_arm_6dof_v2_description/meshes/Forearm_1.stl" scale="0.001 0.001 0.001"/>
-    </geometry>
-    <material name="silver"/>
-  </visual>
-  <collision>
-    <origin rpy="0 0 0" xyz="-0.081402 -0.000774 -0.385994"/>
-    <geometry>
-      <mesh filename="package://mvp_arm_6dof_v2_description/meshes/Forearm_1.stl" scale="0.001 0.001 0.001"/>
-    </geometry>
-  </collision>
-</link>
-<link name="Forearm_Joint_1">
-  <inertial>
-    <origin rpy="0 0 0" xyz="0.019545111524890385 7.79105773380162e-06 -0.00783005977281992"/>
-    <mass value="0.24639014270019174"/>
-    <inertia ixx="6e-05" ixy="-0.0" ixz="8e-06" iyy="9.9e-05" iyz="-0.0" izz="0.000118"/>
-  </inertial>
-  <visual>
-    <origin rpy="0 0 0" xyz="-0.041408 -0.000765 -0.395519"/>
-    <geometry>
-      <mesh filename="package://mvp_arm_6dof_v2_description/meshes/Forearm_Joint_1.stl" scale="0.001 0.001 0.001"/>
-    </geometry>
-    <material name="silver"/>
-  </visual>
-  <collision>
-    <origin rpy="0 0 0" xyz="-0.041408 -0.000765 -0.395519"/>
-    <geometry>
-      <mesh filename="package://mvp_arm_6dof_v2_description/meshes/Forearm_Joint_1.stl" scale="0.001 0.001 0.001"/>
-    </geometry>
-  </collision>
-</link>
-<link name="Servo_Rotator__5__1">
-  <inertial>
-    <origin rpy="0 0 0" xyz="0.00799986632219811 -0.002251236293083818 -5.340036253298486e-06"/>
-    <mass value="0.012286224598738087"/>
-    <inertia ixx="0.0" ixy="-0.0" ixz="-0.0" iyy="1e-06" iyz="-0.0" izz="0.0"/>
-  </inertial>
-  <visual>
-    <origin rpy="0 0 0" xyz="0.020867 -0.0215 -0.354057"/>
-    <geometry>
-      <mesh filename="package://mvp_arm_6dof_v2_description/meshes/Servo_Rotator__5__1.stl" scale="0.001 0.001 0.001"/>
-    </geometry>
-    <material name="silver"/>
-  </visual>
-  <collision>
-    <origin rpy="0 0 0" xyz="0.020867 -0.0215 -0.354057"/>
-    <geometry>
-      <mesh filename="package://mvp_arm_6dof_v2_description/meshes/Servo_Rotator__5__1.stl" scale="0.001 0.001 0.001"/>
-    </geometry>
-  </collision>
-</link>
-<link name="Elbow_Hinge__1__2">
-  <inertial>
-    <origin rpy="0 0 0" xyz="-0.013495411982010678 3.3022629769563494e-15 0.010254437334501432"/>
-    <mass value="0.0037556666472927302"/>
-    <inertia ixx="2e-06" ixy="0.0" ixz="-0.0" iyy="1e-06" iyz="-0.0" izz="1e-06"/>
-  </inertial>
-  <visual>
-    <origin rpy="0 0 0" xyz="-0.000617 -0.0005 -0.327543"/>
-    <geometry>
-      <mesh filename="package://mvp_arm_6dof_v2_description/meshes/Elbow_Hinge__1__2.stl" scale="0.001 0.001 0.001"/>
-    </geometry>
-    <material name="silver"/>
-  </visual>
-  <collision>
-    <origin rpy="0 0 0" xyz="-0.000617 -0.0005 -0.327543"/>
-    <geometry>
-      <mesh filename="package://mvp_arm_6dof_v2_description/meshes/Elbow_Hinge__1__2.stl" scale="0.001 0.001 0.001"/>
-    </geometry>
-  </collision>
-</link>
-<link name="Arm_Link_1">
-  <inertial>
-    <origin rpy="0 0 0" xyz="4.7314773535239024e-05 -0.018999999999999035 0.07720570491989823"/>
-    <mass value="0.21463602179697447"/>
-    <inertia ixx="0.000582" ixy="0.0" ixz="-0.0" iyy="0.000568" iyz="-0.0" izz="3.7e-05"/>
-  </inertial>
-  <visual>
-    <origin rpy="0 0 0" xyz="0.011984 -0.0195 -0.162551"/>
-    <geometry>
-      <mesh filename="package://mvp_arm_6dof_v2_description/meshes/Arm_Link_1.stl" scale="0.001 0.001 0.001"/>
-    </geometry>
-    <material name="silver"/>
-  </visual>
-  <collision>
-    <origin rpy="0 0 0" xyz="0.011984 -0.0195 -0.162551"/>
-    <geometry>
-      <mesh filename="package://mvp_arm_6dof_v2_description/meshes/Arm_Link_1.stl" scale="0.001 0.001 0.001"/>
-    </geometry>
-  </collision>
-</link>
-<link name="Shoulder_Joint_1">
-  <inertial>
-    <origin rpy="0 0 0" xyz="7.287449404962842e-05 0.0016854028904963768 0.013016506375220449"/>
-    <mass value="0.1980303324276481"/>
-    <inertia ixx="0.000259" ixy="-0.0" ixz="-0.0" iyy="0.000259" iyz="-6e-06" izz="0.00042"/>
-  </inertial>
-  <visual>
-    <origin rpy="0 0 0" xyz="0.0 -0.0 -0.131"/>
-    <geometry>
-      <mesh filename="package://mvp_arm_6dof_v2_description/meshes/Shoulder_Joint_1.stl" scale="0.001 0.001 0.001"/>
-    </geometry>
-    <material name="silver"/>
-  </visual>
-  <collision>
-    <origin rpy="0 0 0" xyz="0.0 -0.0 -0.131"/>
-    <geometry>
-      <mesh filename="package://mvp_arm_6dof_v2_description/meshes/Shoulder_Joint_1.stl" scale="0.001 0.001 0.001"/>
-    </geometry>
-  </collision>
-</link>
-<link name="Wrist_Hinge_1">
-  <inertial>
-    <origin rpy="0 0 0" xyz="-0.0006100381163169633 0.020989965286603927 -0.008256993530336987"/>
-    <mass value="0.0037556666472927302"/>
-    <inertia ixx="2e-06" ixy="-0.0" ixz="-0.0" iyy="1e-06" iyz="0.0" izz="1e-06"/>
-  </inertial>
-  <visual>
-    <origin rpy="0 0 0" xyz="-0.222312 0.019985 -0.377955"/>
-    <geometry>
-      <mesh filename="package://mvp_arm_6dof_v2_description/meshes/Wrist_Hinge_1.stl" scale="0.001 0.001 0.001"/>
-    </geometry>
-    <material name="silver"/>
-  </visual>
-  <collision>
-    <origin rpy="0 0 0" xyz="-0.222312 0.019985 -0.377955"/>
-    <geometry>
-      <mesh filename="package://mvp_arm_6dof_v2_description/meshes/Wrist_Hinge_1.stl" scale="0.001 0.001 0.001"/>
-    </geometry>
-  </collision>
-</link>
-<link name="Bracket__1__1">
-  <inertial>
-    <origin rpy="0 0 0" xyz="0.0024261508410601262 9.893036074812322e-06 0.007842544811764884"/>
-    <mass value="0.0016262220015435807"/>
-    <inertia ixx="0.0" ixy="-0.0" ixz="-0.0" iyy="0.0" iyz="-0.0" izz="0.0"/>
-  </inertial>
-  <visual>
-    <origin rpy="0 0 0" xyz="-0.237889 -0.000408 -0.308593"/>
-    <geometry>
-      <mesh filename="package://mvp_arm_6dof_v2_description/meshes/Bracket__1__1.stl" scale="0.001 0.001 0.001"/>
-    </geometry>
-    <material name="silver"/>
-  </visual>
-  <collision>
-    <origin rpy="0 0 0" xyz="-0.237889 -0.000408 -0.308593"/>
-    <geometry>
-      <mesh filename="package://mvp_arm_6dof_v2_description/meshes/Bracket__1__1.stl" scale="0.001 0.001 0.001"/>
-    </geometry>
-  </collision>
-</link>
-<link name="Servo__1__1">
-  <inertial>
-    <origin rpy="0 0 0" xyz="0.021606945197516048 -0.00802128163614104 -0.018110424224670407"/>
-    <mass value="0.32411536495008075"/>
-    <inertia ixx="5e-05" ixy="-0.0" ixz="1e-06" iyy="9.1e-05" iyz="-0.0" izz="7.9e-05"/>
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
Commit message: Update mvp_arm_6dof_v2.xacro

File: mvp_arm_6dof_v2_description/urdf/mvp_arm_6dof_v2.xacro (robot description, xacro)
@@ -464,5 +464,5 @@
   </collision>
 </link>
-<link name="Left_Servo_Finger_Connector_1">
+<!-- <link name="Left_Servo_Finger_Connector_1">
   <inertial>
     <origin rpy="0 0 0" xyz="0.0001409165693066483 0.010442814922828104 -0.0009679780292277673"/>
@@ -503,25 +503,5 @@
     </geometry>
   </collision>
-</link>
-<link name="Right_Gripper_Finger_1">
-  <inertial>
-    <origin rpy="0 0 0" xyz="0.00023279382761542955 0.006324368095181814 -0.01118969345139914"/>
-    <mass value="0.00839361387509603"/>
-    <inertia ixx="1e-06" ixy="-0.0" ixz="-0.0" iyy="2e-06" iyz="0.0" izz="1e-06"/>
-  </inertial>
-  <visual>
-    <origin rpy="0 0 0" xyz="-0.279016 0.031028 -0.301575"/>
-    <geometry>
-      <mesh filename="package://mvp_arm_6dof_v2_description/meshes/Right_Gripper_Finger_1.stl" scale="0.001 0.001 0.001"/>
-    </geometry>
-    <material name="silver"/>
-  </visual>
-  <collision>
-    <origin rpy="0 0 0" xyz="-0.279016 0.031028 -0.301575"/>
-    <geometry>
-      <mesh filename="package://mvp_arm_6dof_v2_description/meshes/Right_Gripper_Finger_1.stl" scale="0.001 0.001 0.001"/>
-    </geometry>
-  </collision>
-</link>
+</link> -->
 <link name="Right_Gripper_Finger_1">
   <inertial>
@@ -541,24 +521,4 @@
     <geometry>
       <mesh filename="package://mvp_arm_6dof_v2_description/meshes/Right_Gripper_Finger_1.stl" scale="0.001 0.001 0.001"/>
-    </geometry>
-  </collision>
-</link>
-<link name="Left_Gripper_Finger_1">
-  <inertial>
-    <origin rpy="0 0 0" xyz="0.020268338652761286 -0.013192067636801953 -0.011636448396533217"/>
-    <mass value="0.008393613874943608"/>
-    <inertia ixx="1e-06" ixy="0.0" ixz="-0.0" iyy="2e-06" iyz="-0.0" izz="1e-06"/>
-  </inertial>
-  <visual>
-    <origin rpy="0 0 0" xyz="-0.258959 -0.033792 -0.302581"/>
-    <geometry>
-      <mesh filename="package://mvp_arm_6dof_v2_description/meshes/Left_Gripper_Finger_1.stl" scale="0.001 0.001 0.001"/>
-    </geometry>
-    <material name="silver"/>
-  </visual>
-  <collision>
-    <origin rpy="0 0 0" xyz="-0.258959 -0.033792 -0.302581"/>
-    <geometry>
-      <mesh filename="package://mvp_arm_6dof_v2_description/meshes/Left_Gripper_Finger_1.stl" scale="0.001 0.001 0.001"/>
     </geometry>
   </collision>
@@ -701,5 +661,5 @@
   <child link="Gripper_Slider_1"/>
 </joint>
-<joint name="Rev8" type="continuous">
+<!-- <joint name="Rev8" type="continuous">
   <origin rpy="0 0 0" xyz="-0.000161 0.008051 -0.004438"/>
   <parent link="Servo_Rotator__1__1"/>
@@ -719,4 +679,10 @@
   <axis xyz="0.020917 0.012351 -0.999705"/>
 </joint>
+<joint name="Rev11" type="continuous">
+  <origin rpy="0 0 0" xyz="0.000472 0.020867 -0.001965"/>
+  <parent link="Left_Servo_Finger_Connector_1"/>
+  <child link="Left_Gripper_Finger_1"/>
+  <axis xyz="0.020917 0.012351 -0.999705"/>
+</joint> -->
 <joint name="Slider1" type="prismatic">
   <origin rpy="0 0 0" xyz="0.051083 -0.022409 -0.0056"/>
@@ -724,5 +690,5 @@
   <child link="Right_Gripper_Finger_1"/>
   <axis xyz="-0.000474 0.999924 0.012343"/>
-  <limit effort="100" lower="0.0" upper="0.0" velocity="100"/>
+  <limit effort="100" lower="0.0" upper=".0150" velocity="100"/>
 </joint>
 <joint name="Slider2" type="prismatic">
@@ -731,11 +697,5 @@
   <child link="Left_Gripper_Finger_1"/>
   <axis xyz="-0.000474 0.999924 0.012343"/>
-  <limit effort="100" lower="0.0" upper="0.0" velocity="100"/>
-</joint>
-<joint name="Rev11" type="continuous">
-  <origin rpy="0 0 0" xyz="0.000472 0.020867 -0.001965"/>
-  <parent link="Left_Servo_Finger_Connector_1"/>
-  <child link="Left_Gripper_Finger_1"/>
-  <axis xyz="0.020917 0.012351 -0.999705"/>
+  <limit effort="100" lower="-.0150" upper="0" velocity="100"/>
 </joint>
 </robot>
